File: design.kicad_sch (KiCad schematic)
At the start: 4 parts, among them J1 USB_C_Receptacle

Commit message: ?
Parts:
- added J3: Conn_01x03, Connector:Pogo-Pin-01x03_2.54, symbol Connector_Generic:Conn_01x03
- added U?: CH340G, Package_SO:SOIC-16_3.9x9.9mm_P1.27mm, symbol Interface_USB:CH340G
- R1, R2: renamed from R?; footprint (none) -> Resistor_SMD:R_0805_2012Metric
- gave numbers to parts that had none: 1
Changed lines of the file:
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@@
   (symbol (lib_id "Connector:USB_C_Receptacle") (at 259.08 62.23 180) (unit 1)
     (in_bom yes) (on_board yes)
-    (property "Reference" "J?" (id 0) (at 256.3622 94.4118 0))
+    (property "Reference" "J2" (id 0) (at 256.3622 94.4118 0))
     (property "Value" "USB_C_Receptacle" (id 1) (at 256.3622 92.1004 0))
     (property "Footprint" "Connector_USB:USB_C_Receptacle_HRO_TYPE-C-31-M-12" (id 2) (at 255.27 62.23 0)
@@
   (symbol (lib_id "power:GND") (at 34.925 92.71 0) (unit 1)
     (in_bom yes) (on_board yes)
-    (property "Reference" "#PWR?" (id 0) (at 34.925 99.06 0)
+    (property "Reference" "#PWR0102" (id 0) (at 34.925 99.06 0)
       (effects (font (size 1.27 1.27)) hide)
     )
@@
   (symbol (lib_id "power:VCC") (at 56.515 26.67 0) (unit 1)
     (in_bom yes) (on_board yes)
-    (property "Reference" "#PWR?" (id 0) (at 56.515 30.48 0)
+    (property "Reference" "#PWR0103" (id 0) (at 56.515 30.48 0)
       (effects (font (size 1.27 1.27)) hide)
     )
@@
   (symbol (lib_id "Device:R_Small") (at 63.5 31.75 270) (unit 1)
     (in_bom yes) (on_board yes)
-    (property "Reference" "R?" (id 0) (at 63.5 26.7716 90))
+    (property "Reference" "R1" (id 0) (at 63.5 26.7716 90))
     (property "Value" "R_Small" (id 1) (at 63.5 29.083 90))
-    (property "Footprint" "" (id 2) (at 63.5 31.75 0)
+    (property "Footprint" "Resistor_SMD:R_0805_2012Metric" (id 2) (at 63.5 31.75 0)
       (effects (font (size 1.27 1.27)) hide)
     )
@@
   (symbol (lib_id "Device:R_Small") (at 72.39 34.29 270) (unit 1)
     (in_bom yes) (on_board yes)
-    (property "Reference" "R?" (id 0) (at 72.39 29.3116 90))
+    (property "Reference" "R2" (id 0) (at 72.39 29.3116 90))
     (property "Value" "R_Small" (id 1) (at 72.39 31.623 90))
-    (property "Footprint" "" (id 2) (at 72.39 34.29 0)
+    (property "Footprint" "Resistor_SMD:R_0805_2012Metric" (id 2) (at 72.39 34.29 0)
       (effects (font (size 1.27 1.27)) hide)
     )
@@
   (symbol (lib_id "power:GND") (at 80.01 34.29 0) (unit 1)
     (in_bom yes) (on_board yes)
-    (property "Reference" "#PWR?" (id 0) (at 80.01 40.64 0)
+    (property "Reference" "#PWR0101" (id 0) (at 80.01 40.64 0)
       (effects (font (size 1.27 1.27)) hide)
     )
@@
     (pin "1")
   )
+  (symbol (lib_id "Connector_Generic:Conn_01x03") (at 189.23 53.34 0) (unit 1)
+    (in_bom yes) (on_board yes) (fields_autoplaced)
+    (property "Reference" "J3" (id 0) (at 191.77 52.0699 0)
+      (effects (font (size 1.27 1.27)) (justify left))
+    )
+    (property "Value" "Conn_01x03" (id 1) (at 191.77 54.6099 0)
+      (effects (font (size 1.27 1.27)) (justify left))
+    )
+    (property "Footprint" "Connector:Pogo-Pin-01x03_2.54" (id 2) (at 189.23 53.34 0)
+      (effects (font (size 1.27 1.27)) hide)
+    )
+    (property "Datasheet" "~" (id 3) (at 189.23 53.34 0)
+      (effects (font (size 1.27 1.27)) hide)
+    )
+    (pin "1")
+    (pin "2")
+    (pin "3")
+  )
+  (symbol (lib_id "Interface_USB:CH340G") (at 123.19 50.8 0) (unit 1)
+    (in_bom yes) (on_board yes) (fields_autoplaced)
+    (property "Reference" "U?" (id 0) (at 125.2094 66.04 0)
+      (effects (font (size 1.27 1.27)) (justify left))
+    )
+    (property "Value" "CH340G" (id 1) (at 125.2094 68.58 0)
+      (effects (font (size 1.27 1.27)) (justify left))
+    )
+    (property "Footprint" "Package_SO:SOIC-16_3.9x9.9mm_P1.27mm" (id 2) (at 124.46 64.77 0)
+      (effects (font (size 1.27 1.27)) (justify left) hide)
+    )
+    (property "Datasheet" "http://www.datasheet5.com/pdf-local-2195953" (id 3) (at 114.3 30.48 0)
+      (effects (font (size 1.27 1.27)) hide)
+    )
+    (pin "1")
+    (pin "10")
+    (pin "11")
+    (pin "12")
+    (pin "13")
+    (pin "14")
+    (pin "15")
+    (pin "16")
+    (pin "2")
+    (pin "3")
+    (pin "4")
+    (pin "5")
+    (pin "6")
+    (pin "7")
+    (pin "8")
+    (pin "9")
+  )
   (sheet_instances
     (path "/" (page "1"))
   )
   (symbol_instances
+    (path "/00000000-0000-0000-0000-000061c9a95a"
+      (reference "#PWR0101") (unit 1) (value "GND") (footprint "")
+    )
     (path "/00000000-0000-0000-0000-000061c96041"
-      (reference "#PWR?") (unit 1) (value "GND") (footprint "")
+      (reference "#PWR0102") (unit 1) (value "GND") (footprint "")
     )
     (path "/00000000-0000-0000-0000-000061c96e6b"
-      (reference "#PWR?") (unit 1) (value "VCC") (footprint "")
-    )
-    (path "/00000000-0000-0000-0000-000061c9a95a"
-      (reference "#PWR?") (unit 1) (value "GND") (footprint "")
+      (reference "#PWR0103") (unit 1) (value "VCC") (footprint "")
     )
     (path "/00000000-0000-0000-0000-0000616f374e"
@@
     )
     (path "/00000000-0000-0000-0000-000061c9239b"
-      (reference "J?") (unit 1) (value "USB_C_Receptacle") (footprint "Connector_USB:USB_C_Receptacle_HRO_TYPE-C-31-M-12")
+      (reference "J2") (unit 1) (value "USB_C_Receptacle") (footprint "Connector_USB:USB_C_Receptacle_HRO_TYPE-C-31-M-12")
+    )
+    (path "/25165c40-f1cb-4a81-ad74-6bea9e79eda2"
+      (reference "J3") (unit 1) (value "Conn_01x03") (footprint "Connector:Pogo-Pin-01x03_2.54")
     )
     (path "/00000000-0000-0000-0000-000061c988f5"
-      (reference "R?") (unit 1) (value "R_Small") (footprint "")
+      (reference "R1") (unit 1) (value "R_Small") (footprint "Resistor_SMD:R_0805_2012Metric")
     )
     (path "/00000000-0000-0000-0000-000061c99361"
-      (reference "R?") (unit 1) (value "R_Small") (footprint "")
+      (reference "R2") (unit 1) (value "R_Small") (footprint "Resistor_SMD:R_0805_2012Metric")
+    )
+    (path "/5058348c-32f3-4102-a4e4-1e82f2768116"
+      (reference "U?") (unit 1) (value "CH340G") (footprint "Package_SO:SOIC-16_3.9x9.9mm_P1.27mm")
     )
   )

Commit message: delete titel block
Other:
- title: <<project_name>> -> (none)
Changed lines of the file:
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@@
 (kicad_sch (version 20211123) (generator eeschema)
   (paper "A4")
-  (title_block
-    (title "<<project_name>>")
-    (date "<<date>>")
-    (rev "<<hash>>")
-  )
   (junction (at 80.01 34.29) (diameter 0) (color 0 0 0 0)
   )
